File: Klipper_Expander/KiCad/STM32_Klipper_Expander.sch (KiCad schematic (older format))
At the start: 45 parts, among them J1 USB_B_Micro, J10 Conn_01x01, J11 Conn_01x03, J12 Conn_01x02, J2 Conn_01x04, J4 Conn_01x03, J5 Vin, J6 Screw_Terminal_01x08, J7 Conn_01x02, J8 Conn_01x02, J9 Conn_01x02, Q1 IRLML6344TRPBF, Q2 IRLML6344TRPBF, Q3 IRLML6344TRPBF, Q4 IRLML6344TRPBF, SW2 SW_SPST, U1 STM32F042F6Px, U2 AP2127K-3.3, U3 74LVC1G17

Commit message: Klipper Expander V2 (#9)
* Status LED's and silkscren adjustments.

Added status LED's for Vin (12/24V), USB (5V), and all 4 mosfets on the drain. LED's will signal mosfet output status.

Gerber and PNP files still need to be completed.

* Updated README to include fuse purchasing options for 2,5,and 10A fuses as well as an assortment.

* Updated Gerber and Production files, Minor changes

Changed thermsitor pullups to 4K7 to increse range and reliability.
Added silkscreen to indicate what the status LED's are showing.

* Conifg and Step additions

Changed onboard LED on PA4 to become a "
Status" LED that will turn on when board is powered and connected.
Parts:
- added D2, D3, D4, D5, D6, D7: LED, LED_SMD:LED_0805_2012Metric, symbol Device:LED
- added R15, R18, R19, R20, R22: 4.7K, Resistor_SMD:R_0805_2012Metric, symbol Device:R
- added R21: 1K, Resistor_SMD:R_0805_2012Metric, symbol Device:R
- J12: value Conn_01x02 -> Conn_01x03; footprint Connector_PinHeader_2.54mm:PinHeader_1x02_P2.54mm_Vertical -> Connector_PinHeader_2.54mm:PinHeader_1x03_P2.54mm_Vertical; symbol Connector_Generic:Conn_01x02 -> Connector_Generic:Conn_01x03
- R16, R17: value 10K -> 4.7K; LCSC C17414 -> C17673; MPN RC0805JR-0710KL -> RC0805JR-074K7L; SKU 301010361 -> 301010306
- U3: footprint Package_TO_SOT_SMD:SOT-353_SC-70-5 -> digikey-footprints:SOT-753; LCSC C124293 -> C6076; MPN 74LVC1G17SE-7 -> (none)
Connections:
- wire segments 140 -> 168
