File: SKR-Mini_Screen_Adaptor/V3.0/Kicad/SKR-Mini_Screen.kicad_pcb (KiCad board)
At the start: 2 copper layers, 22.9 x 43.2 mm, 6 parts, among them J1 Board_EXP1, J2 Board_SPI, J3 Screen_EXP1, J4 Screen_EXP2

Commit message: Update header pin spacing
 - Update header pin spacing from 0.75 to 1mm to aid in fit for some shrouded headers
 - Update project to KiCad 6.0
Other:
- rule pad_to_mask_clearance: 0.051 -> 0
Changed lines of the file:
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@@
   )
   (setup
-    (pad_to_mask_clearance 0.051)
-    (solder_mask_min_width 0.25)
+    (stackup
+      (layer "F.SilkS" (type "Top Silk Screen"))
+      (layer "F.Paste" (type "Top Solder Paste"))
+      (layer "F.Mask" (type "Top Solder Mask") (thickness 0.01))
+      (layer "F.Cu" (type "copper") (thickness 0.035))
+      (layer "dielectric 1" (type "core") (thickness 1.51) (material "FR4") (epsilon_r 4.5) (loss_tangent 0.02))
+      (layer "B.Cu" (type "copper") (thickness 0.035))
+      (layer "B.Mask" (type "Bottom Solder Mask") (thickness 0.01))
+      (layer "B.Paste" (type "Bottom Solder Paste"))
+      (layer "B.SilkS" (type "Bottom Silk Screen"))
+      (copper_finish "None")
+      (dielectric_constraints no)
+    )
+    (pad_to_mask_clearance 0)
     (grid_origin 125.73 106.68)
     (pcbplotparams
