File: Daylight/Disco_on_a_stick/Daylight_Disco.kicad_pcb (KiCad board)
At the start: 2 copper layers, 270 x 11 mm, 41 parts, among them J1 Conn_01x03_Male, J2 Conn_01x01_Male, J3 Conn_01x01_Male

Commit message: Daylight | Add output connectors to the RGB sticks
Provided pick and place files for all varieties as well.
Created individual README.md files with BOM and changelog.
Parts:
- J2: value Conn_01x01_Male -> Conn_01x03_Male; footprint Daylight:PinHeader-1-with-SMDpad -> Daylight:JST_XH_S3B-XH-A-1_1x03_P2.50mm_Horizontal
- moved J2 9.73 mm to (263.2, 30.5), turned to -90 degrees
Connections:
- J2 pad 1: DOUT -> GND
Routing:
- net +5V: track 23.7 -> 41.4 mm, vias 3 -> 5
- net Net-(D17-Pad2): track 11.0 -> 18.0 mm, vias 0 -> 2
- net DOUT: track 255.4 -> 261.5 mm, vias 0 -> 1
- net GND: vias 34 -> 38
Other:
- board text added: "Disco on a stick v1.1 by Blamm"
- board text added: "GND 5V DOUT"
- board text removed: "Disco on a stick v1.0 by Blamm"
