File: V0_Display_RP2040/KiCad/V0_Display.kicad_pcb (KiCad board)
At the start: 2 copper layers, 80 x 35 mm, 47 parts, among them J2 I2C Header 1, J3 SWD, J4 USB_B_Micro, J5 GPIO, J7 USB_Header, J8 Conn_01x02, SW1 RESET, SW5 BOOTSEL, SW6 Killswitch, SW7 Rotary_Encoder_Switch, U1 AP2127K-3.3, U2 USBLC6-2P6, U3 74LVC1G17, U4 W25Q16JVUXIQ_TR, U5 RP2040, Y1 12Mhz

Commit message: Clean up
Parts:
- C1, C2: footprint Voron0 2040 display:C_0603_1608Metric -> Library:C_0603_1608Metric
- C10, C11, C12, C13, C14, C15, C16, C17, C3, C4, C5, C6, C7, C8, C9: footprint Voron0 2040 display:C_0402_1005Metric -> Library:C_0402_1005Metric
- D1: footprint Voron0 2040 display:LED_WS2812B_PLCC4_5.0x5.0mm_P3.2mm -> Library:LED_WS2812B_PLCC4_5.0x5.0mm_P3.2mm
- H1, H2, H3, H4: footprint Voron0 2040 display:MountingHole_3.2mm_M3 -> Library:MountingHole_3.2mm_M3
- J3: footprint Voron0 2040 display:PinHeader_1x05_P2.54mm_Vertical -> Library:PinHeader_1x05_P2.54mm_Vertical
- J7: footprint Voron0 2040 display:PinHeader_1x04_P2.54mm_Vertical -> Library:PinHeader_1x04_P2.54mm_Vertical
- J8: footprint Voron0 2040 display:PinHeader_1x02_P2.54mm_Vertical -> Library:PinHeader_1x02_P2.54mm_Vertical
- L1: footprint Voron0 2040 display:L_0402_1005Metric -> Library:L_0402_1005Metric
- R1, R3, R4, R9: footprint Voron0 2040 display:R_0603_1608Metric -> Library:R_0603_1608Metric
- R2: footprint Voron0 2040 display:R_0402_1005Metric -> Library:R_0603_1608Metric
- R7, R8: footprint Voron0 2040 display:R_0402_1005Metric -> Library:R_0402_1005Metric
- SW7: footprint Voron0 2040 display:EN11_Encoder -> Library:EN11_Encoder
- U1: footprint Voron0 2040 display:SOT-23-5 -> Library:SOT-23-5
- U2: footprint Voron0 2040 display:SOT-666 -> Library:SOT-666
- U3: footprint Voron0 2040 display:SOT-753 -> Library:SOT-753
- U4: footprint Voron0 2040 display:IC_W25Q16JVUXIQ_TR -> Library:IC_W25Q16JVUXIQ_TR
- U5: footprint Voron0 2040 display:RP2040-QFN-56 -> Library:RP2040-QFN-56
- Y1: footprint Voron0 2040 display:Crystal_SMD_3225-4Pin_3.2x2.5mm -> Library:Crystal_SMD_3225-4Pin_3.2x2.5mm
- moved J8 7.77 mm to (153.7, 59.8)
- moved C4 3.55 mm to (127.1, 60.4)
- moved Y1 3.07 mm to (124.5, 60.8)
- moved C3 2.89 mm to (121.6, 60.0)
- moved R2 2.03 mm to (120.8, 61.8), turned to 0 degrees
Routing:
- net Net-(D1-DOUT): track 14.1 -> 6.33 mm
- net VBUS: track 116.4 -> 122.8 mm
- net OSC_IN: track 5.49 -> 8.92 mm
- net Net-(D1-DIN): track 39.7 -> 41.9 mm
- net Net-(C4-Pad1): track 6.59 -> 8.00 mm
- net OSC_OUT: track 2.65 -> 3.90 mm
- net Kill_Switch: track 69.0 -> 69.6 mm
- net GND: track 93.4 -> 94.0 mm
Other:
- rule pad_to_mask_clearance: 0.05 -> 0

Commit message: Fixed up gerbers
Parts:
- moved H5 6.99 mm to (131.0, 66.5)
Other:
- board text added: "GPIO"
