File: V0_Display_RP2040/KiCad/V0_Display_RP2040.kicad_pcb (KiCad board)
At the start: 2 copper layers, 80 x 35 mm, 47 parts, among them J2 I2C Header 1, J3 SWD, J4 USB_B_Micro, J5 GPIO, J7 USB_Header, J8 Conn_01x02, SW1 RESET, SW5 BOOTSEL, SW6 Killswitch, SW7 Rotary_Encoder_Switch, U1 AP2127K-3.3, U2 USBLC6-2P6, U3 74LVC1G17, U4 W25Q16JVUXIQ_TR, U5 RP2040, Y1 12Mhz

Commit message: Updated silkscreen
Other:
- board text added: "V0-2040 Display V1 by th0mpy"
- board text removed: "V0-2040 Display V1"
